Commit message: fix the controller and add scripts for dependency

File: Diff_H80_description/urdf/materials.xacro (robot description, xacro)
@@ -1,6 +1,6 @@
-<?xml version="1.0" ?>
-<robot name="Diff_H80" xmlns:xacro="http://www.ros.org/wiki/xacro" >
-<material name="silver">
-  <color rgba="0.700 0.700 0.700 1.000"/>
-</material>
+<?xml version="1.0"?>
+<robot name="Diff_H80" xmlns:xacro="http://www.ros.org/wiki/xacro">
+  <material name="silver">
+    <color rgba="0.700 0.700 0.700 1.000" />
+  </material>
 </robot>
